Commit message: updates to robot urdf structure, added ignore missing reports cuz annoying

File: src/robot/urdf/robot_fin.urdf (robot description, URDF)
Before this commit: robot robot_model, 20 links, 19 joints
Links:
- link face_panel_link: geometry collision box size=0.12 0.18 0.01; visual box size=0.12 0.18 0.01

File: src/robot/urdf/torso.xacro (robot description, xacro)
@@ -31,7 +31,7 @@
 		<link name="face_panel_link">
 			<visual>
-				<origin xyz="${torso_length / 2.0 + face_panel_length / 2.0} 0 ${torso_height / 4.0}" rpy="0 0 0" />
+				<origin xyz="${torso_length / 2.0 - face_panel_height / 2.0} 0 ${torso_height / 2.0 + face_panel_length / 2.0}" rpy="0 0 0" />
 				<geometry>
-					<box size="${face_panel_length} ${face_panel_width} ${face_panel_height}" />
+					<box size="${face_panel_height} ${face_panel_width} ${face_panel_length}" />
 				</geometry>
 				<material name="face_black">
@@ -40,15 +40,15 @@
 			</visual>
 			<collision>
-				<origin xyz="${torso_length / 2.0 + face_panel_length / 2.0} 0 ${torso_height / 4.0}" rpy="0 0 0" />
+				<origin xyz="${torso_length / 2.0 - face_panel_height / 2.0} 0 ${torso_height / 2.0 + face_panel_length / 2.0}" rpy="0 0 0" />
 				<geometry>
-					<box size="${face_panel_length} ${face_panel_width} ${face_panel_height}" />
+					<box size="${face_panel_height} ${face_panel_width} ${face_panel_length}" />
 				</geometry>
 			</collision>
 			<xacro:box_inertial_from_mass
-				l="${face_panel_length}"
+				l="${face_panel_height}"
 				w="${face_panel_width}"
-				h="${face_panel_height}"
+				h="${face_panel_length}"
 				mass="${face_panel_mass}"
-				origin_xyz="${torso_length / 2.0 + face_panel_length / 2.0} 0 ${torso_height / 4.0}" />
+				origin_xyz="${torso_length / 2.0 - face_panel_height / 2.0} 0 ${torso_height / 2.0 + face_panel_length / 2.0}" />
 		</link>
 		<joint name="face_panel_joint" type="fixed">
