Commit message: arm controllers, world scene, object models

File: src/robot/urdf/controller.xacro (robot description, xacro)
@@ -26,4 +26,58 @@
         <state_interface name="velocity"/>
       </joint>
+      <joint name="left_arm_shoulder_joint">
+        <command_interface name="position"/>
+        <command_interface name="effort">
+          <param name="min">-10.0</param>
+          <param name="max">10.0</param>
+        </command_interface>
+        <state_interface name="position"/>
+        <state_interface name="velocity"/>
+      </joint>
+      <joint name="left_arm_elbow_joint">
+        <command_interface name="position"/>
+        <command_interface name="effort">
+          <param name="min">-10.0</param>
+          <param name="max">10.0</param>
+        </command_interface>
+        <state_interface name="position"/>
+        <state_interface name="velocity"/>
+      </joint>
+      <joint name="right_arm_shoulder_joint">
+        <command_interface name="position"/>
+        <command_interface name="effort">
+          <param name="min">-10.0</param>
+          <param name="max">10.0</param>
+        </command_interface>
+        <state_interface name="position"/>
+        <state_interface name="velocity"/>
+      </joint>
+      <joint name="right_arm_elbow_joint">
+        <command_interface name="position"/>
+        <command_interface name="effort">
+          <param name="min">-10.0</param>
+          <param name="max">10.0</param>
+        </command_interface>
+        <state_interface name="position"/>
+        <state_interface name="velocity"/>
+      </joint>
+      <joint name="left_arm_wrist_joint">
+        <command_interface name="position"/>
+        <command_interface name="effort">
+          <param name="min">-5.0</param>
+          <param name="max">5.0</param>
+        </command_interface>
+        <state_interface name="position"/>
+        <state_interface name="velocity"/>
+      </joint>
+      <joint name="right_arm_wrist_joint">
+        <command_interface name="position"/>
+        <command_interface name="effort">
+          <param name="min">-5.0</param>
+          <param name="max">5.0</param>
+        </command_interface>
+        <state_interface name="position"/>
+        <state_interface name="velocity"/>
+      </joint>
     </ros2_control>
   </xacro:macro>
