Commit message: fixed lidar and camera publishing issue, created world with a big room

File: src/robot/urdf/car_constants.xacro (robot description, xacro)
@@ -4,8 +4,8 @@
 	<xacro:property name="chassis_width" value="0.42" />
 	<xacro:property name="chassis_height" value="0.2" />
-	<xacro:property name="chassis_mass" value="0.4" />
+	<xacro:property name="chassis_mass" value="3.5" />
 	<xacro:property name="wheel_radius" value="0.10" />
 	<xacro:property name="wheel_width" value="0.04" />
-	<xacro:property name="wheel_mass" value="1.2" />
+	<xacro:property name="wheel_mass" value="0.8" />
 	<xacro:property name="wheel_x_offset" value="0.17" />
 	<xacro:property name="wheel_y_offset" value="0.23" />

File: src/robot/urdf/robot_chasis.xacro (robot description, xacro)
@@ -31,4 +31,5 @@
 			<axis xyz="0 1 0"/>
 			<dynamics damping="0.2" friction="0.1"/>
+			<limit effort="20.0" velocity="15.0"/>
 		</joint>
 	</xacro:macro>

Commit message: updates to run file

File: src/robot/urdf/car_constants.xacro (robot description, xacro)
@@ -3,5 +3,5 @@
 	<xacro:property name="chassis_length" value="0.52" />
 	<xacro:property name="chassis_width" value="0.42" />
-	<xacro:property name="chassis_height" value="0.2" />
+	<xacro:property name="chassis_height" value="0.1" />
 	<xacro:property name="chassis_mass" value="3.5" />
 	<xacro:property name="wheel_radius" value="0.10" />
@@ -12,5 +12,5 @@
 	<xacro:property name="torso_length" value="0.52" />
 	<xacro:property name="torso_width" value="0.42" />
-	<xacro:property name="torso_height" value="0.2" />
+	<xacro:property name="torso_height" value="0.1" />
 	<xacro:property name="torso_mass" value="6.0" />
 	<xacro:property name="torso_z_offset" value="${chassis_height / 2.0 + torso_height / 2.0}" />

File: src/robot/urdf/gazebo.xacro (robot description, xacro)
@@ -4,6 +4,9 @@
 		<gazebo reference="${link_name}">
 			<material>Gazebo/DarkGrey</material>
-			<mu1>1.2</mu1>
-			<mu2>1.2</mu2>
+			<fdir1>1 0 0</fdir1>
+			<mu1>1.1</mu1>
+			<mu2>0.2</mu2>
+			<slip1>0.0</slip1>
+			<slip2>0.25</slip2>
 			<kp>1000000.0</kp>
 			<kd>100.0</kd>
