Commit message: EKF + SLAM drift correction

File: src/robot/urdf/gazebo.xacro (robot description, xacro)
@@ -7,6 +7,4 @@
 			<mu1>2.0</mu1>
 			<mu2>1.5</mu2>
-			<slip1>0.0</slip1>
-			<slip2>0.03</slip2>
 			<kp>1000000.0</kp>
 			<kd>100.0</kd>
@@ -57,4 +55,5 @@
 				<visualize>true</visualize>
 				<topic>scan</topic>
+				<gz_frame_id>lidar_link</gz_frame_id>
 				<ray>
 					<scan>
@@ -80,4 +79,14 @@
 			</sensor>
 		</gazebo>
+		<gazebo reference="imu_link">
+			<selfCollide>false</selfCollide>
+			<sensor name="torso_imu" type="imu">
+				<always_on>true</always_on>
+				<update_rate>50</update_rate>
+				<visualize>false</visualize>
+				<topic>imu/data_raw</topic>
+				<gz_frame_id>imu_link</gz_frame_id>
+			</sensor>
+		</gazebo>
 		<gazebo>
 			<plugin filename="libgz_ros2_control-system.so"

File: src/robot/urdf/sensors.xacro (robot description, xacro)
@@ -55,4 +55,31 @@
 			<origin xyz="0 0 ${torso_height / 2.0 + 0.04}" rpy="0 0 0" />
 		</joint>
+		<link name="imu_link">
+			<visual>
+				<origin xyz="0 0 0" rpy="0 0 0" />
+				<geometry>
+					<sphere radius="0.03" />
+				</geometry>
+				<material name="imu_gray">
+					<color rgba="0.3 0.3 0.3 1.0"/>
+				</material>
+			</visual>
+			<collision>
+				<origin xyz="0 0 0" rpy="0 0 0" />
+				<geometry>
+					<sphere radius="0.03" />
+				</geometry>
+			</collision>
+			<xacro:box_inertial_from_mass
+				l="0.06"
+				w="0.06"
+				h="0.06"
+				mass="0.1" />
+		</link>
+		<joint name="imu_joint" type="fixed">
+			<parent link="${parent}"/>
+			<child link="imu_link"/>
+			<origin xyz="0 0 ${chassis_height / 2.0 + 0.08}" rpy="0 0 0" />
+		</joint>
 	</xacro:macro>
 </robot>
